File: board/board.kicad_pcb (KiCad board)
At the start: 2 copper layers, 45 x 13 mm, 34 parts, among them J1 Conn_01x02_Pin, J2 Conn_01x02_Pin, J3 003_power, U1 TPS65131

Commit message: initial b146
Parts:
- removed C10, C13, C14, C15, C16, C17, C18, C9: 22uF, Capacitor_SMD:C_0805_2012Metric
- removed C11: 10pF, Capacitor_SMD:C_0402_1005Metric
- removed C12: 220nF, Capacitor_SMD:C_0402_1005Metric
- removed D2: SS12, Diode_SMD:D_SMA
- removed J2: Conn_01x02_Pin, Connector_PinHeader_2.54mm:PinHeader_1x02_P2.54mm_Vertical
- removed L2: 4.7uH, Inductor_SMD:L_6.3x6.3_H3
- removed NT1: NetTie_2, NetTie:NetTie-2_SMD_Pad0.5mm
- removed R5: 82k, Resistor_SMD:R_0402_1005Metric
- removed R6: 1M, Resistor_SMD:R_0402_1005Metric
- removed R7: 51k, Resistor_SMD:R_0402_1005Metric
- C1: value 22uF -> 1uF; footprint Capacitor_SMD:C_0805_2012Metric -> Capacitor_SMD:C_0603_1608Metric
- C2, C4: value 22uF -> 220uF; footprint Capacitor_SMD:C_0805_2012Metric -> Capacitor_SMD:CP_Elec_10x14.3
- C3: value 22uF -> 100nF; footprint Capacitor_SMD:C_0805_2012Metric -> Capacitor_SMD:C_0603_1608Metric
- C5: footprint Capacitor_SMD:C_0402_1005Metric -> Capacitor_SMD:C_0603_1608Metric
- C6: value 10pF -> 1uF; footprint Capacitor_SMD:C_0402_1005Metric -> Capacitor_SMD:C_1206_3216Metric
- C7: value 10nF -> 100nF; footprint Capacitor_SMD:C_0402_1005Metric -> Capacitor_SMD:C_0603_1608Metric
- C8: value 4.7nF -> 1uF; footprint Capacitor_SMD:C_0402_1005Metric -> Capacitor_SMD:C_0603_1608Metric
- D1: value SS12 -> PMEG6010EP,115; footprint Diode_SMD:D_SMA -> Diode_SMD:D_SOD-128
- L1: value 4.7uH -> 47uH; footprint Inductor_SMD:L_6.3x6.3_H3 -> Inductor_SMD:L_Sunlord_MWSA1206S-470
- R1: value 100R -> 100k
- R2: value 1M -> 100k; footprint Resistor_SMD:R_0402_1005Metric -> Resistor_SMD:R_0603_1608Metric
- R3: value 100k -> 2.5k; footprint Resistor_SMD:R_0402_1005Metric -> Resistor_SMD:R_0603_1608Metric
- U1: value TPS65131 -> XL6019E1; footprint Package_DFN_QFN:VQFN-24-1EP_4x4mm_P0.5mm_EP2.45x2.45mm_ThermalVias -> Package_TO_SOT_SMD:TO-263-5_TabPin3
- moved J1 38.2 mm to (180.0, 111.8), turned to 90 degrees
- moved C4 28.2 mm to (178.9, 98.8), turned to -90 degrees
- moved LOGO1 25.9 mm to (175.7, 115.4)
- moved C6 24.4 mm to (181.1, 106.7)
- moved C3 22.8 mm to (170.4, 111.1), turned to -90 degrees
- moved C2 19.2 mm to (145.6, 110.1), turned to -90 degrees
- moved R3 18.0 mm to (170.6, 107.0), turned to -90 degrees
- moved C5 17.2 mm to (180.4, 108.6), turned to 180 degrees
- moved C8 17.0 mm to (147.4, 96.0), turned to 180 degrees
- moved C7 15.9 mm to (147.4, 97.5), turned to 180 degrees
- moved U1 15.6 mm to (157.9, 110.3), turned to 180 degrees
- moved R2 14.0 mm to (170.6, 104.0), turned to -90 degrees
- moved C1 13.6 mm to (171.9, 111.1), turned to -90 degrees
- moved D1 12.6 mm to (168.4, 97.2), turned to 180 degrees
- moved R1 10.9 mm to (168.9, 111.1), turned to -90 degrees
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Connections:
- C4 pad 1: /DCDC/5V -> /DCDC/+out
- C5 pad 1: Net-(U1-ENN) -> /DCDC/+out
- C5 pad 2: /DCDC/GNDA -> GND
- C6 pad 1: Net-(U1-FBP) -> /DCDC/+out
- C6 pad 2: /DCDC/+out -> GND
- C7 pad 1: /DCDC/GNDA -> /DCDC/5V
- C7 pad 2: Net-(U1-CP) -> GND
- C8 pad 1: /DCDC/GNDA -> /DCDC/5V
- C8 pad 2: Net-(U1-CN) -> GND
- R1 pad 2: Net-(U1-ENN) -> Net-(U1-EN)
- R2 pad 2: Net-(U1-FBP) -> Net-(U1-FB)
- R3 pad 1: Net-(U1-FBP) -> Net-(U1-FB)
- R3 pad 2: /DCDC/GNDA -> GND
- U1 pad 1: Net-(D1-A) -> GND
- U1 pad 2: GND -> Net-(U1-EN)
- U1 pad 3: GND -> Net-(D1-A)
- U1 pad 4: Net-(U1-ENN) -> /DCDC/5V
- U1 pad 5: /DCDC/5V -> Net-(U1-FB)
Routing:
- net GND: track 38.7 -> 93.6 mm, vias 27 -> 32
- net /DCDC/5V: track 35.1 -> 63.5 mm
- net /DCDC/-out: track 26.7 -> 0.00 mm
- net Net-(D2-K): track 17.3 -> 0.00 mm
- net /DCDC/+out: track 24.3 -> 41.4 mm, vias 1 -> 0
- net /DCDC/GNDA: track 16.1 -> 0.00 mm, vias 2 -> 0
- net Net-(U1-ENN): track 10.8 -> 0.00 mm, vias 2 -> 0
- net Net-(D1-A): track 17.9 -> 26.9 mm
- net Net-(U1-FB): track 0.00 -> 6.70 mm
- net Net-(U1-FBN): track 4.79 -> 0.00 mm
- net Net-(U1-FBP): track 3.65 -> 0.00 mm
- net Net-(U1-EN): track 0.00 -> 3.39 mm
- net Net-(U1-VREF): track 3.12 -> 0.00 mm
- net Net-(U1-CN): track 2.02 -> 0.00 mm
- net Net-(U1-CP): track 1.68 -> 0.00 mm
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Other:
- board size 45 x 13 mm -> 45 x 29 mm
- board text added: "osf.b146.v1.0"
- board text removed: "osf.b145.v1.0"
