File: board/board.kicad_sch (KiCad schematic)
At the start: 4 parts, among them J1 Conn_01x02_Pin, J2 Conn_01x02_Pin, J3 003_power

Commit message: initial b146
Parts:
- removed J2: Conn_01x02_Pin, Connector_PinHeader_2.54mm:PinHeader_1x02_P2.54mm_Vertical, symbol Connector:Conn_01x02_Pin
Other:
- sheet DCDC ports: added none; removed -out
Changed lines of the file:
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@@
   (junction (at 182.88 129.54) (diameter 0) (color 0 0 0 0)
-  )
-  (junction (at 182.88 116.84) (diameter 0) (color 0 0 0 0)
   )
   (no_connect (at 120.65 138.43))
@@
     (stroke (width 0) (type default))
   )
-  (wire (pts (xy 175.26 119.38) (xy 184.15 119.38))
-    (stroke (width 0) (type default))
-  )
   (wire (pts (xy 175.26 110.49) (xy 184.15 110.49))
     (stroke (width 0) (type default))
@@
     (stroke (width 0) (type default))
   )
-  (wire (pts (xy 182.88 116.84) (xy 184.15 116.84))
-    (stroke (width 0) (type default))
-  )
   (wire (pts (xy 182.88 107.95) (xy 184.15 107.95))
-    (stroke (width 0) (type default))
-  )
-  (wire (pts (xy 182.88 116.84) (xy 182.88 107.95))
     (stroke (width 0) (type default))
   )
@@
     (stroke (width 0) (type default))
   )
-  (wire (pts (xy 182.88 129.54) (xy 182.88 116.84))
+  (wire (pts (xy 182.88 107.95) (xy 182.88 129.54))
     (stroke (width 0) (type default))
   )
@@
         (path "/57732dd3-1162-4c3f-88bd-31bf473d124d"
           (reference "J3") (unit 1)
-        )
-      )
-    )
-  )
-  (symbol (lib_id "Connector:Conn_01x02_Pin") (at 189.23 116.84 0) (mirror y) (unit 1)
-    (in_bom yes) (on_board yes) (dnp no) (fields_autoplaced)
-    (property "Reference" "J2" (at 190.5 116.84 0)
-      (effects (font (size 1.27 1.27)) (justify right))
-    )
-    (property "Value" "Conn_01x02_Pin" (at 190.5 119.38 0)
-      (effects (font (size 1.27 1.27)) (justify right))
-    )
-    (property "Footprint" "Connector_PinHeader_2.54mm:PinHeader_1x02_P2.54mm_Vertical" (at 189.23 116.84 0)
-      (effects (font (size 1.27 1.27)) hide)
-    )
-    (property "Datasheet" "~" (at 189.23 116.84 0)
-      (effects (font (size 1.27 1.27)) hide)
-    )
-    (pin "1")
-    (pin "2")
-    (instances
-      (project "board"
-        (path "/57732dd3-1162-4c3f-88bd-31bf473d124d"
-          (reference "J2") (unit 1)
         )
       )
@@
       (effects (font (size 1.27 1.27)) (justify right))
     )
-    (pin "-out" input (at 175.26 119.38 0)
-      (effects (font (size 1.27 1.27)) (justify right))
-    )
